File: hardware/pi-interface/pi-interface.sch (KiCad schematic (older format))
At the start: 8 parts, among them J1 RasPI_IO_Header, P1 SL030 RFID, P2 Molex HDD Power, P3 Door Solenoid, Q1 BC237

Commit message: Improved PCB, still needs checking against parts ordered
Parts:
- removed RL1: RM50-xx11, Relays_ThroughHole:Relay_SPDS_OMRON-G6E, symbol RM50-xx11
- added RLY1: RELAY_HJR-3FF_Z, w_relay:relay_hjr-3ff_z, symbol RELAY_HJR-3FF_Z
- J1: Farnell Part (none) -> 1098052
- P2: Farnell Part (none) -> 148086
- P3: Farnell Part (none) -> 2396251
- R1: value R -> 220R
Connections:
- wire segments 37 -> 38
Changed lines of the file:
@@
 F 2 "Socket_Strips:Socket_Strip_Straight_2x13" H 4950 2450 60  0001 C CNN
 F 3 "" H 4950 2450 60  0000 C CNN
+F 4 "1098052" H 4950 2450 60  0001 C CNN "Farnell Part"
 	1    4950 2450
 	1    0    0    -1
-$EndComp
-$Comp
-L RM50-xx11 RL1
-U 1 1 55E0CBF6
-P 6700 2550
-F 0 "RL1" H 7150 2700 50  0000 L CNN
-F 1 "RM50-xx11" H 7150 2600 50  0000 L CNN
-F 2 "Relays_ThroughHole:Relay_SPDS_OMRON-G6E" H 6700 2550 60  0001 C CNN
-F 3 "" H 6700 2550 60  0000 C CNN
-	1    6700 2550
-	1    0    0    1
 $EndComp
 $Comp
@@
 F 3 "" H 3400 2100 60  0000 C CNN
 	1    3400 2100
-	-1   0    0    -1
+	-1   0    0    1
 $EndComp
 $Comp
@@
 F 2 "w_conn_screw:mstba_2,5%2f2-g-5,08" H 7450 2000 60  0001 C CNN
 F 3 "" H 7450 2000 60  0000 C CNN
+F 4 "2396251" H 7450 2000 60  0001 C CNN "Farnell Part"
 	1    7450 2000
-	1    0    0    -1
+	1    0    0    1
 $EndComp
 $Comp
@@
 F 2 "w_conn_pc:conn_hdd_15-24-4449" H 6450 1600 60  0001 C CNN
 F 3 "" H 6450 1600 60  0000 C CNN
+F 4 "148086" H 6450 1600 60  0001 C CNN "Farnell Part"
 	1    6450 1600
 	0    -1   -1   0
@@
 P 5950 3100
 F 0 "R1" V 6030 3100 50  0000 C CNN
-F 1 "R" V 5950 3100 50  0000 C CNN
+F 1 "220R" V 5950 3100 50  0000 C CNN
 F 2 "Resistors_ThroughHole:Resistor_Horizontal_RM10mm" V 5880 3100 30  0001 C CNN
 F 3 "" H 5950 3100 30  0000 C CNN
@@
 	6300 1850 5750 1850
 Wire Wire Line
-	6400 1800 6400 2050
-Wire Wire Line
-	6400 2050 5750 2050
-Wire Wire Line
 	6600 1800 6600 1950
 Wire Wire Line
 	5750 2850 5950 2850
 Wire Wire Line
-	4000 3550 6500 3550
+	4000 3550 7050 3550
 Wire Wire Line
 	4000 3550 4000 3050
@@
 	6150 2850 6150 2700
 Wire Wire Line
-	6500 2850 6500 3150
+	6500 2750 6500 3150
 Wire Wire Line
 	5950 2850 5950 2950
@@
 	6600 1950 7250 1950
 Wire Wire Line
-	7250 2050 7250 3000
+	7250 3000 7250 2050
 Wire Wire Line
-	7250 3000 7000 3000
-Wire Wire Line
-	7000 3000 7000 2850
-Wire Wire Line
-	6900 2250 6900 2150
-Wire Wire Line
-	6900 2150 6500 2150
+	6800 3000 7250 3000
 Connection ~ 6300 2250
 Connection ~ 6300 1850
+$Comp
+L RELAY_HJR-3FF_Z RLY1
+U 1 1 55EC4E47
+P 6650 2550
+F 0 "RLY1" H 6650 2800 60  0000 C CNN
+F 1 "RELAY_HJR-3FF_Z" H 6650 2315 60  0000 C CNN
+F 2 "w_relay:relay_hjr-3ff_z" H 6650 2550 60  0000 C CNN
+F 3 "" H 6650 2550 60  0000 C CNN
+F 4 "2325631" H 6650 2550 60  0001 C CNN "Farnell Part"
+	1    6650 2550
+	0    -1   1    0
+$EndComp
+Wire Wire Line
+	6500 2150 6750 2150
+Wire Wire Line
+	6750 2150 6750 2350
+Wire Wire Line
+	6500 2250 6500 2350
+Connection ~ 6500 2850
+Wire Wire Line
+	6800 2750 6800 3000
+Wire Wire Line
+	6400 1800 7050 1800
+Wire Wire Line
+	7050 1800 7050 3550
+Connection ~ 6500 3550
 $EndSCHEMATC

Commit message: First finished (fingers crossed) PCB design.
Parts:
- P2: footprint w_conn_pc:conn_hdd_15-24-4449 -> w_conn_screw:mstbva_2,5%2f4-g-5,08
Changed lines of the file:
@@
 F 0 "P2" H 6450 1850 50  0000 C CNN
 F 1 "Molex HDD Power" V 6550 1600 50  0000 C CNN
-F 2 "w_conn_pc:conn_hdd_15-24-4449" H 6450 1600 60  0001 C CNN
+F 2 "w_conn_screw:mstbva_2,5%2f4-g-5,08" H 6450 1600 60  0001 C CNN
 F 3 "" H 6450 1600 60  0000 C CNN
 F 4 "148086" H 6450 1600 60  0001 C CNN "Farnell Part"

Commit message: I2S DAC added to PCB.  Fixes #17
Also added DoES Liverpool logo to silkscreen, and other mods for the first revision of the PCB sent to be manufactured.
Parts:
- removed J1: RasPI_IO_Header, Socket_Strips:Socket_Strip_Straight_2x13, symbol RasPI_IO_Header
- added J1: Raspberry_Pi_2_3, Pin_Headers:Pin_Header_Straight_2x20, symbol Raspberry_Pi_2_3
- added U1: MAX98357A-Breakout, MCQN Ltd:MAX98357-Breakout, symbol MAX98357A-Breakout
Connections:
- wire segments 38 -> 43
- no-connect marks 0 -> 5
Other:
- moved on the sheet: P1, R1
Changed lines of the file:
@@
 LIBS:w_transistor
 LIBS:w_relay
+LIBS:MCQN-Schematic-Components
 LIBS:pi-interface-cache
-EELAYER 25 0
+EELAYER 26 0
 EELAYER END
 $Descr A4 11693 8268
@@
 $EndDescr
 $Comp
-L RasPI_IO_Header J1
-U 1 1 55E0CB24
-P 4950 2450
-F 0 "J1" H 4950 3150 60  0000 C CNN
-F 1 "RasPI_IO_Header" H 4950 1750 60  0000 C CNN
-F 2 "Socket_Strips:Socket_Strip_Straight_2x13" H 4950 2450 60  0001 C CNN
-F 3 "" H 4950 2450 60  0000 C CNN
-F 4 "1098052" H 4950 2450 60  0001 C CNN "Farnell Part"
-	1    4950 2450
-	1    0    0    -1
-$EndComp
-$Comp
 L CONN_01X06 P1
 U 1 1 55E0CC33
-P 3400 2100
-F 0 "P1" H 3400 2450 50  0000 C CNN
-F 1 "SL030 RFID" V 3500 2100 50  0000 C CNN
-F 2 "Pin_Headers:Pin_Header_Angled_1x06" H 3400 2100 60  0001 C CNN
-F 3 "" H 3400 2100 60  0000 C CNN
-	1    3400 2100
+P 1900 2300
+F 0 "P1" H 1900 2650 50  0000 C CNN
+F 1 "SL030 RFID" V 2000 2300 50  0000 C CNN
+F 2 "Pin_Headers:Pin_Header_Angled_1x06" H 1900 2300 60  0001 C CNN
+F 3 "" H 1900 2300 60  0000 C CNN
+	1    1900 2300
 	-1   0    0    1
 $EndComp
@@
 L R R1
 U 1 1 55EB05B7
-P 5950 3100
-F 0 "R1" V 6030 3100 50  0000 C CNN
-F 1 "220R" V 5950 3100 50  0000 C CNN
-F 2 "Resistors_ThroughHole:Resistor_Horizontal_RM10mm" V 5880 3100 30  0001 C CNN
-F 3 "" H 5950 3100 30  0000 C CNN
-	1    5950 3100
-	1    0    0    -1
+P 5950 3350
+F 0 "R1" V 6030 3350 50  0000 C CNN
+F 1 "220R" V 5950 3350 50  0000 C CNN
+F 2 "Resistors_ThroughHole:Resistor_Horizontal_RM10mm" V 5880 3350 30  0001 C CNN
+F 3 "" H 5950 3350 30  0000 C CNN
+	1    5950 3350
+	0    1    1    0
 $EndComp
 $Comp
@@
 	1    0    0    -1
 $EndComp
-Wire Wire Line
-	3600 1850 4150 1850
-Wire Wire Line
-	3600 2050 3700 2050
-Wire Wire Line
-	3700 2050 3700 1950
-Wire Wire Line
-	3700 1950 4150 1950
-Wire Wire Line
-	3600 2150 3750 2150
-Wire Wire Line
-	3750 2150 3750 2050
-Wire Wire Line
-	3750 2050 4150 2050
-Wire Wire Line
-	3600 2250 3800 2250
-Wire Wire Line
-	3800 2250 3800 2150
-Wire Wire Line
-	3800 2150 4150 2150
-Wire Wire Line
-	3600 2350 3850 2350
-Wire Wire Line
-	3850 2350 3850 2250
-Wire Wire Line
-	3850 2250 4150 2250
-Wire Wire Line
-	6300 1800 6300 2250
-Wire Wire Line
-	6300 1850 5750 1850
-Wire Wire Line
-	6600 1800 6600 1950
-Wire Wire Line
-	5750 2850 5950 2850
-Wire Wire Line
-	4000 3550 7050 3550
-Wire Wire Line
-	4000 3550 4000 3050
-Wire Wire Line
-	4000 3050 4150 3050
-Wire Wire Line
-	6500 1800 6500 2150
-Wire Wire Line
-	6150 2400 6150 2250
-Wire Wire Line
-	6150 2250 6500 2250
-Wire Wire Line
-	6500 2850 6150 2850
-Wire Wire Line
-	6150 2850 6150 2700
-Wire Wire Line
-	6500 2750 6500 3150
-Wire Wire Line
-	5950 2850 5950 2950
-Wire Wire Line
-	5950 3250 5950 3350
-Wire Wire Line
-	5950 3350 6200 3350
-Wire Wire Line
-	6600 1950 7250 1950
-Wire Wire Line
-	7250 3000 7250 2050
-Wire Wire Line
-	6800 3000 7250 3000
-Connection ~ 6300 2250
-Connection ~ 6300 1850
 $Comp
 L RELAY_HJR-3FF_Z RLY1
@@
 	0    -1   1    0
 $EndComp
+$Comp
+L MAX98357A-Breakout U1
+U 1 1 598F2091
+P 5300 3350
+F 0 "U1" H 5300 4437 60  0000 C CNN
+F 1 "MAX98357A-Breakout" H 5300 4331 60  0000 C CNN
+F 2 "MCQN Ltd:MAX98357-Breakout" H 5300 3350 60  0001 C CNN
+F 3 "" H 5300 3350 60  0001 C CNN
+	1    5300 3350
+	1    0    0    -1
+$EndComp
+NoConn ~ 5800 2800
+NoConn ~ 5800 2900
+$Comp
+L Raspberry_Pi_2_3 J1
+U 1 1 598F91EF
+P 3400 3150
+F 0 "J1" H 3400 4628 50  0000 C CNN
+F 1 "Raspberry_Pi_2_3" H 3400 4537 50  0000 C CNN
+F 2 "Pin_Headers:Pin_Header_Straight_2x20" H 4400 4400 50  0001 C CNN
+F 3 "" H 3450 3000 50  0001 C CNN
+	1    3400 3150
+	-1   0    0    -1
+$EndComp
+NoConn ~ 2100 2150
+NoConn ~ 4800 2950
+NoConn ~ 4800 2850
+Wire Wire Line
+	6300 1800 6300 2250
+Wire Wire Line
+	6600 1800 6600 1950
+Wire Wire Line
+	6500 1800 6500 2150
+Wire Wire Line
+	6150 2400 6150 2250
+Wire Wire Line
+	6150 2250 6500 2250
+Wire Wire Line
+	6500 2850 6150 2850
+Wire Wire Line
+	6150 2850 6150 2700
+Wire Wire Line
+	6500 2750 6500 3150
+Wire Wire Line
+	6600 1950 7250 1950
+Wire Wire Line
+	7250 3000 7250 2050
+Wire Wire Line
+	6800 3000 7250 3000
+Connection ~ 6300 2250
 Wire Wire Line
 	6500 2150 6750 2150
@@
 	6400 1800 7050 1800
 Wire Wire Line
-	7050 1800 7050 3550
+	7050 1800 7050 4550
 Connection ~ 6500 3550
+Wire Wire Line
+	2200 1800 2200 2050
+Wire Wire Line
+	2200 2050 2100 2050
+Wire Wire Line
+	2500 2250 2100 2250
+Wire Wire Line
+	2500 2350 2100 2350
+Wire Wire Line
+	2500 2450 2100 2450
+Wire Wire Line
+	2100 2550 2200 2550
+Wire Wire Line
+	2200 2550 2200 4550
+Wire Wire Line
+	6200 3350 6100 3350
+Wire Wire Line
+	4300 3350 5800 3350
+Wire Wire Line
+	6500 4550 6500 3550
+Wire Wire Line
+	4800 2550 4500 2550
+Wire Wire Line
+	4500 2550 4500 2750
+Wire Wire Line
+	4500 2750 4300 2750
+Wire Wire Line
+	4800 2650 4300 2650
+Wire Wire Line
+	4800 2750 4600 2750
+Wire Wire Line
+	4600 2750 4600 2950
+Wire Wire Line
+	4600 2950 4300 2950
+Wire Wire Line
+	4800 3150 4400 3150
+Wire Wire Line
+	4400 3150 4400 1850
+Wire Wire Line
+	4800 3050 4700 3050
+Wire Wire Line
+	4700 3050 4700 4550
+Wire Wire Line
+	3700 4450 3700 4550
+Wire Wire Line
+	2200 4550 7050 4550
+Connection ~ 3700 4550
+Connection ~ 4700 4550
+Connection ~ 6500 4550
+Wire Wire Line
+	2200 1800 3300 1800
+Wire Wire Line
+	3300 1800 3300 1850
+Wire Wire Line
+	3600 1850 6300 1850
+Connection ~ 4400 1850
+Connection ~ 6300 1850
 $EndSCHEMATC

Commit message: Enlarge holes for the Molex connector.  Fixes #21
Parts:
- P2: symbol CONN_01X04 -> CONN_01X04-RESCUE-pi-interface
Changed lines of the file:
@@
 EESchema Schematic File Version 2
+LIBS:pi-interface-rescue
 LIBS:power
 LIBS:device
@@
 $EndComp
 $Comp
-L CONN_01X04 P2
+L CONN_01X04-RESCUE-pi-interface P2
 U 1 1 55E0DD9F
 P 6450 1600

Commit message: Add Farnell part numbers for more of the components. Part of #6
Parts:
- D1: Farnell Part (none) -> 2675047
- J1: Farnell Part (none) -> 3419290
- Q1: Farnell Part (none) -> 1574377
- R1: Farnell Part (none) -> 1700228
Changed lines of the file:
@@
 F 2 "Resistors_ThroughHole:Resistor_Horizontal_RM10mm" V 5880 3350 30  0001 C CNN
 F 3 "" H 5950 3350 30  0000 C CNN
+F 4 "1700228" V 5950 3350 60  0001 C CNN "Farnell Part"
 	1    5950 3350
 	0    1    1    0
@@
 F 2 "Diodes_ThroughHole:Diode_DO-201AD_Horizontal_RM15" H 6150 2550 60  0001 C CNN
 F 3 "" H 6150 2550 60  0000 C CNN
+F 4 "2675047" H 6150 2550 60  0001 C CNN "Farnell Part"
 	1    6150 2550
 	0    1    1    0
@@
 F 2 "Transistors_TO-220:TO-220_Neutral123_Vertical_LargePads" H 6600 3275 50  0000 L CIN
 F 3 "" H 6400 3350 50  0000 L CNN
+F 4 "1574377" H 6400 3350 60  0001 C CNN "Farnell Part"
 	1    6400 3350
 	1    0    0    -1
@@
 F 2 "Pin_Headers:Pin_Header_Straight_2x20" H 4400 4400 50  0001 C CNN
 F 3 "" H 3450 3000 50  0001 C CNN
+F 4 "3419290" H 3400 3150 60  0001 C CNN "Farnell Part"
 	1    3400 3150
 	-1   0    0    -1
